File: eagle/v0.2/M.2 SoM breakout board v0.2-Placement-03011.brd (EAGLE design)
At the start: 140 x 120 mm, 154 parts, among them J10 CON_122_SMD_HEADER, J11 WAFER-HY2.0-4PWB, J12 TP_OPEN, J13 SIM-NANO-4FF, J15 CON_122_SMD_HEADER, J19 TP_OPEN, J2 DCJ0202, J20 TP_OPEN, J21 SIP-2, J22 SIP-2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

Commit message: Update M.2 SoM breakout board v0.2-Placement-03011.brd
update
Parts:
- moved U1 15.9 mm to (38.7, 107.3), turned to 90 degrees
- moved R2 15.5 mm to (39.4, 109.6), turned to 0 degrees
- moved R7 12.9 mm to (37.4, 109.6), turned to 180 degrees
- moved R18 0.51 mm to (35.9, 107.0)
- moved R74 0.51 mm to (34.9, 107.0)
Routing:
- net SDA: track 313.0 -> 218.1 mm
- net !RESET: track 219.7 -> 148.2 mm
- net PWM0: track 259.7 -> 228.3 mm
- net GPIO1: track 256.6 -> 234.8 mm
- net VUSB-MCU: track 63.7 -> 44.7 mm
- net TS: track 62.3 -> 45.4 mm
- net VBAT: track 76.8 -> 65.5 mm
- net VCC: track 74.7 -> 66.1 mm
- net SCL: track 284.1 -> 277.6 mm
- net VIN: track 44.4 -> 39.8 mm
- net 5VDC: track 6.60 -> 2.74 mm
- net ADC6: track 127.5 -> 123.9 mm
- net REGN: track 40.2 -> 37.0 mm
- net GND: track 140.1 -> 138.0 mm
- net VBUS: track 3.62 -> 2.46 mm
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