File: eagle/v0.2-layout/M.2 SoM breakout board v0.2.brd (EAGLE design)
At the start: 140 x 120 mm, 155 parts, among them J10 CON_122_SMD_HEADER, J11 WAFER-HY2.0-4PWB, J12 TP_OPEN, J13 SIM-NANO-4FF, J15 CON_122_SMD_HEADER, J19 TP_OPEN, J2 DCJ0202, J20 TP_OPEN, J21 SIP-2, J22 SIP-2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

Commit message: Upadte
update layout
Parts:
- removed J14: (no value), particle-studios:1X03
- removed R17: 10K, Particle:R0402_B
- added 3V3, GND, GND15, VBAT, VCC, VIN: (no value), particle-studios:S2751-46R
- added J8: TP_OPEN, particle SZ:TP_OPEN
- added R32: nc, particle SZ:R-0402S
- added R33: 1K, RedBear:R-0402S
- added TP1: TPTPEB, particle SZ:TPEB
- Q3, Q5: value IR6401 -> HSS2333
- Q4: value IRLML6401 -> HSS2333
- R21: value 1M -> 1M/NC
- R22: value 1K -> 10K; device Particle:R0402_B -> particle-studios:R0603_P
- moved R22 2.60 mm to (12.1, 106.3), turned to 180 degrees
- moved D2 1.75 mm to (33.8, 109.1), turned to 180 degrees
- moved D17 0.38 mm to (-11.9, 101.4)
- moved J22 0.32 mm to (59.7, 114.5), turned to 270 degrees
- moved R37 0.18 mm to (-18.4, 3.87)
- moved LED3 0.18 mm to (41.9, 101.5)
- moved R13 0.18 mm to (39.4, 101.5)
- moved R18 0.13 mm to (35.3, 106.4)
Connections:
- new net N$13: R18.1, R32.1, R74.2
- new net N$14: J8.2, R32.2
- new net N$20: R33.1, S4.1, S4.4
- net +3V3: now also 3V3.1; no longer R22.2
- net ADC7: now also TP1.1; no longer J14.1
- net CS: no longer J14.2
- net GND: now also GND.1, GND15.1, R22.1, S4.3, S4.6; no longer R17.1, S4.2, S4.5
- net GPIO0: no longer J14.3
- net N$300: now also R33.2
- net N$302: now also S4.2, S4.5; no longer S4.3, S4.6
- net N$57: now also R22.2; no longer R17.2
- net N$7: no longer R22.1
- net TS: now also J8.1; no longer R18.1, R74.2
- net VBAT: now also VBAT.1
- net VCC: now also VCC.1
- net VIN: now also VIN.1
Routing:
- net N$20: track 0.00 -> 14.4 mm, vias 0 -> 1
- net ADC7: track 134.6 -> 125.0 mm
- net +3V3: track 531.8 -> 537.6 mm, vias 44 -> 43
- net CS: track 165.3 -> 159.9 mm, vias 4 -> 5
- net PWM3: track 234.2 -> 230.1 mm
- net N$13: track 0.00 -> 4.01 mm, vias 0 -> 1
- net N$302: track 16.2 -> 19.9 mm
- net GPIO0: track 192.2 -> 188.8 mm
- net VUSBMCU: track 83.3 -> 86.4 mm
- net TS: track 45.9 -> 42.8 mm
- net N$7: track 15.9 -> 12.8 mm
- net GND: track 261.1 -> 263.7 mm, vias 656 -> 663
- net N$14: track 0.00 -> 1.31 mm
- net VUSB-MCU: track 54.9 -> 53.6 mm
- net N$301: track 13.5 -> 14.2 mm
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