File: eagle/v0.2-layout/M.2 SoM breakout board v0.2.sch (EAGLE design)
At the start: 155 parts, among them J10 CON_122_SMD_HEADER, J11 WAFER-HY2.0-4PWB, J12 TP_OPEN, J13 SIM-NANO-4FF, J15 CON_122_SMD_HEADER, J19 TP_OPEN, J2 DCJ0202, J20 TP_OPEN, J21 SIP-2, J22 SIP-2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

Commit message: Upadte
update layout
Parts:
- removed J14: (no value), particle-studios:CONN_03
- removed R17: 10K, Particle:R-US_
- added 3V3, GND, GND15, VBAT, VCC, VIN: TP-S2751-46R, particle-studios:TP-S2751-46R
- added J8: TP_OPEN, particle SZ:TP_OPEN
- added R32: nc, particle SZ:RES0402S
- added R33: 1K, RedBear:RES0402S
- added TP1: TPTPEB, particle SZ:TPTPEB
- Q3, Q5: value IR6401 -> HSS2333
- Q4: value IRLML6401 -> HSS2333
- R21: value 1M -> 1M/NC
- R22: value 1K -> 10K; device Particle:R-US_ -> particle-studios:RES_10K_0603
Connections:
- new net N$13: R18.1, R32.1, R74.2
- new net N$14: J8.2, R32.2
- new net N$20: R33.1, S4.1, S4.4
- net +3V3: now also 3V3.TP; no longer R22.2
- net ADC7: now also TP1.1; no longer J14.1
- net CS: no longer J14.2
- net GND: now also GND.TP, GND15.TP, R22.1, S4.3, S4.6; no longer R17.1, S4.2, S4.5
- net GPIO0: no longer J14.3
- net N$300: now also R33.2
- net N$302: now also S4.2, S4.5; no longer S4.3, S4.6
- net N$57: now also R22.2; no longer R17.2
- net N$7: no longer R22.1
- net TS: now also J8.1; no longer R18.1, R74.2
- net VBAT: now also VBAT.TP
- net VCC: now also VCC.TP
- net VIN: now also VIN.TP
Other:
- note added: "16 ADC6:!FUEL_INT"
- note added: "1:change placement"
- note added: "23 Reserve for reset power module"
- note added: "24 Indicate Power status"
- note added: "25 Power enable pin"
- note added: "2:change power module size and pin define place"
- note added: "3:modify sch of the Q3&Q5 to vbat on/off"
- note added: "4: Reserved PG pull-up resistance"
- note added: "5:Add three pin :Charge pin，REGN pin"
- note removed: "12"
- note removed: "15 ADC6:!FUEL_INT"
- note removed: "22 Reserve for reset power module"
- note removed: "23 Indicate Power status"
- note removed: "24 Power enable pin"
- note removed: "Add three pin :Charge pin，REGN pin"
- note removed: "change placement"
- note removed: "modify sch of the Q3&Q5 to vbat on/off"
- moved on the sheet: J21, R22, R30, R74
