File: eagle/V0.3/M.2 SoM breakout board v0.3.brd (EAGLE design)
At the start: 140 x 122 mm, 189 parts, among them J1 3-PIN SMD, J11 WAFER-HY2.0-4PWB, J12 TP_OPEN, J13 SIM-NANO-4FF, J18 PARTICLE-STUDIOS_M_SERIES_M.2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, J19 TP_OPEN, J2 DCJ0202, J20 TP_OPEN, J21 SIP-2, J22 SIP-2, J3 SPARK_CON_30X2_SMD, J5 SCREW-HOLE-3.7, J6 PARTICLE-SZ_PARTICLE-POWER-MO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, J7 SCREW-HOLE-3.7, Q1 HSS2333, Q3 HSS2333, Q4 HSS2333, Q5 HSS2333, T1 TP_SHORT, U1 XC8107, U2 AT24CS64-SSHM-B, U7 NC, X1 BU-SMA-G, X2 BU-SMA-G, X3 BU-SMA-G

Commit message: update
update
Parts:
- removed TP10, TP11, TP12, TP13, TP14, TP15, TP16, TP17, TP18, TP19, TP20, TP21, TP22, TP23, TP24, TP25, TP26, TP27, TP28, TP29, TP3, TP30, TP31, TP32, TP33, TP34, TP35, TP36, TP37, TP38, TP39, TP4, TP40, TP41, TP42, TP43, TP44, TP45, TP46, TP47, TP48, TP49, TP50, TP51, TP52, TP53, TP54, TP57, TP6, TP7, TP9: TPSB1,27, testpad:B1,27
- moved JP4 0.61 mm to (60.7, 19.9)
Connections:
- net !MODE: no longer TP35.TP
- net !RESET: no longer TP36.TP
- net 3V3_AUX: no longer TP30.TP
- net ADC0: no longer TP6.TP
- net ADC1: no longer TP7.TP
- net ADC2: no longer TP9.TP
- net ADC3: no longer TP10.TP
- net ADC4: no longer TP12.TP
- net ADC5: no longer TP13.TP
- net ADC7: no longer TP15.TP
- net CS: no longer TP41.TP
- net CTS: no longer TP39.TP
- net GND: no longer TP11.TP, TP16.TP, TP29.TP, TP45.TP
- net GPIO0: no longer TP48.TP
- net GPIO1: no longer TP49.TP
- net LED_BLUE: no longer TP24.TP
- net LED_GREEN: no longer TP23.TP
- net LED_RED: no longer TP22.TP
- net MISO: no longer TP42.TP
- net MOSI: no longer TP43.TP
- net N$15: no longer TP14.TP
- net NFC1: no longer TP3.TP
- net NFC2: no longer TP4.TP
- net PWM0: no longer TP50.TP
- net PWM1: no longer TP51.TP
- net PWM2: no longer TP52.TP
- net PWM3: no longer TP53.TP
- net RTS: no longer TP40.TP
- net RX: no longer TP38.TP
- net SCK: no longer TP44.TP
- net SCL: no longer TP33.TP
- net SDA: no longer TP34.TP
- net SOM10: no longer TP31.TP
- net SOM11: no longer TP32.TP
- net SOM12: no longer TP46.TP
- net SOM13: no longer TP47.TP
- net SOM14: no longer TP17.TP
- net SOM15: no longer TP18.TP
- net SOM16: no longer TP19.TP
- net SOM17: no longer TP20.TP
- net SOM18: no longer TP21.TP
- net SOM5: no longer TP25.TP
- net SOM6: no longer TP26.TP
- net SOM7: no longer TP27.TP
- net SOM8: no longer TP28.TP
- net SOM9: no longer TP57.TP
- net TX: no longer TP37.TP
- net VCC: no longer TP54.TP
Routing:
- net GND: track 533.7 -> 627.6 mm, vias 613 -> 677
- net VCC: track 128.7 -> 120.0 mm
- net CTS: track 78.9 -> 71.9 mm
- net SCL: track 262.9 -> 256.2 mm
- net SDA: track 268.3 -> 264.0 mm
- net PWM1: track 188.7 -> 184.5 mm, vias 6 -> 5
- net SOM8: track 109.9 -> 106.2 mm
- net 3V3_AUX: track 280.0 -> 276.4 mm
- net SOM17: track 66.4 -> 63.3 mm, vias 3 -> 2
- net RX: track 124.9 -> 122.2 mm
- net SOM10: track 100.9 -> 98.3 mm
- net SOM18: track 66.0 -> 63.4 mm, vias 3 -> 2
- net SOM5: track 116.0 -> 113.4 mm
- net GPIO0: track 192.4 -> 189.9 mm, vias 6 -> 5
- net ADC7: track 55.4 -> 52.9 mm, vias 3 -> 2
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- added copper zone on layer 2, net UB_VBUS
- added copper zone on layer 2, net VUSB
Other:
- board text added: "202404011"
- board text removed: "20240404"

Commit message: update
update
Parts:
- removed J22: SIP-2, particle SZ:SIP-2
- moved JP4 15.8 mm to (60.7, 4.16), turned to 270 degrees
Connections:
- removed net VUSBMCU: J18.16, J22.1
- net CTS: now also JP25.2
- net GPIO1: no longer JP25.2
- net VUSB-MCU: now also J18.16; no longer J22.2
Routing:
- net CTS: track 71.9 -> 176.1 mm, vias 2 -> 4
- net VUSBMCU: track 88.0 -> 0.00 mm
- net GPIO1: track 207.4 -> 123.7 mm, vias 5 -> 2
- net VUSB-MCU: track 51.8 -> 122.3 mm, vias 6 -> 12
- net ADC6: track 119.7 -> 137.5 mm
- net N$15: track 13.0 -> 4.41 mm
- net GND: track 627.6 -> 634.3 mm, vias 677 -> 730
- net +3V3: track 365.7 -> 363.1 mm
- net CHG: track 7.00 -> 9.03 mm
- net TX: track 124.6 -> 125.5 mm
- net RX: track 122.2 -> 122.9 mm
- net !RESET: track 276.7 -> 277.3 mm
- added copper zone on layer 15, net 3V3_AUX
- added copper zone on layer 15, net UB_VBUS1
- added copper zone on layer 15, net VBAT
- added copper zone on layer 15, net VCC
- added copper zone on layer 15, net VIN
- added copper zone on layer 15, net VUSB-MCU
- removed copper zone on layer 15, net +3V3
Other:
- board text added: "20240411"
- board text added: "FEATHERWING"
- board text added: "RGB"
- board text removed: "202404011"
- board text removed: "ADC0"
- board text removed: "ADC1"
- board text removed: "ADC2"
- board text removed: "ADC3"
- board text removed: "ADC4"
- board text removed: "ADC5"
- board text removed: "FEATHER"
- board text removed: "GPIO1"
- board text removed: "J22"

Commit message: update
1.Repair the silk screen to the jumper,change the size of the circle at the position of the small rubber pad
2.Remove the jumper from LED1 to 3V3,R16/NC,R17/NC.R11/NC, R22 as 0R ,make the circuit simple that used DC power supply directly  control, change the  Q1  as nmos and NC reserved
3.Optimize SPI traces to make them equal in length
Parts:
- removed T1: TP_SHORT, particle SZ:TP_SHORT
- D16: value BZT52C3V9 -> PZ3D4V2H; device Diodes:SOD-123 -> particle SZ:SOD-323
- F2: device RedBear:R1206 -> RedBear:F0805
- Q1: value HSS2333 -> L2N7002; device RedBear:SOT-23 -> particle SZ:SOT323
- R11: value 100K -> 1K/NC
- R16: value 1K -> 1K/NC
- R17: value 1K -> 100K/NC
- R18: value NC -> 10K
- R22: value NC -> 0R
- RT1, RT2: device particle SZ:R0603 -> particle SZ:R-0603A
- moved JP4 1.45 mm to (60.7, 2.71)
- moved F2 0.78 mm to (49.8, 109.1)
- moved VBAT 0.66 mm to (35.8, 102.1)
- moved Q1 0.15 mm to (22.9, 109.1)
- turned R22 to 90 degrees
- turned LED1 to 90 degrees
- turned R18 to 90 degrees
- turned D16 to 0 degrees
Connections:
- removed net N$14: R16.2, T1.2
- net +3V3: now also R16.1; no longer T1.1
- net GND: now also D16.1, Q1.2; no longer D16.A, Q1.3
- net N$18: now also R16.2; no longer R16.1
- net N$36: now also Q1.3; no longer Q1.2
- net VBUS: now also F2.P$2; no longer F2.2
- net VCC: now also D16.2; no longer D16.C
- net VUSB: now also F2.P$1; no longer F2.1
Routing:
- net 3V3_AUX: track 276.3 -> 286.1 mm, vias 42 -> 44
- net GND: track 634.3 -> 628.3 mm, vias 730 -> 761
- net SCK: track 135.1 -> 138.8 mm, vias 3 -> 4
- net MOSI: track 135.5 -> 138.8 mm, vias 3 -> 4
- net N$14: track 2.59 -> 0.00 mm
- net +3V3: track 363.1 -> 365.1 mm
- net N$15: track 4.41 -> 5.86 mm
- net ADC6: track 137.5 -> 138.5 mm
- net VIN: track 32.9 -> 33.5 mm
- net N$19: track 3.54 -> 4.08 mm
Other:
- board text removed: "D17"
