File: eagle/V0.5/M.2 SoM breakout board v0.5.sch (EAGLE design)
At the start: 135 parts, among them J1 3-PIN SMD, J11 WAFER-HY2.0-4PWB, J12 TP_OPEN, J13 SIM-NANO-4FF, J18 PARTICLE-STUDIOS_M_SERIES_M.2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, J19 TP_OPEN, J2 DCJ0202, J20 TP_OPEN, J21 SIP-2, J3 SPARK_CON_30X2_SMD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

Commit message: Added antenna cable clips
- added antenna cable clips
- moved qr code square to the bottom left
- moved VIN test point away from the clip to avoid accidental shorting
- added GND test point next to VIN test point
Parts:
- added GND18: TP-S2751-46R, particle-studios:TP-S2751-46R
- added X4, X5, X6: S8111-46R, particle-studios:S8111-46R
Connections:
- net GND: now also GND18.TP, X4.C, X5.C, X6.C
Other:
- moved on the sheet: GND15
Changed lines of the file:
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@@
 <drawing>
 <settings>
-<setting alwaysvectorfont="no"/>
+<setting alwaysvectorfont="yes"/>
 <setting verticaltext="up"/>
 </settings>
-<grid distance="0.025" unitdist="inch" unit="inch" style="lines" multiple="1" display="yes" altdistance="0.01" altunitdist="inch" altunit="inch"/>
+<grid distance="0.05" unitdist="inch" unit="inch" style="lines" multiple="1" display="yes" altdistance="0.01" altunitdist="inch" altunit="inch"/>
 <layers>
 <layer number="1" name="Top" color="4" fill="1" visible="no" active="no"/>
@@
 <part name="+3V2" library="supply1" library_urn="urn:adsk.eagle:library:371" deviceset="+3V3" device=""/>
 <part name="J6" library="M.2 SoM breakout board v0.3" deviceset="M.2-SOM-BREAKOUT-BOARD-V0.2-0228_PARTICLE-SZ_PARTICLE-POWER-MODULE" device=""/>
+<part name="X4" library="particle-studios" library_urn="urn:adsk.eagle:library:10700396" deviceset="S8111-46R" device=""/>
+<part name="X5" library="particle-studios" library_urn="urn:adsk.eagle:library:10700396" deviceset="S8111-46R" device=""/>
+<part name="X6" library="particle-studios" library_urn="urn:adsk.eagle:library:10700396" deviceset="S8111-46R" device=""/>
+<part name="U$2" library="microbuilder" deviceset="GND" device=""/>
+<part name="U$3" library="microbuilder" deviceset="GND" device=""/>
+<part name="U$4" library="microbuilder" deviceset="GND" device=""/>
+<part name="GND18" library="particle-studios" library_urn="urn:adsk.eagle:library:10700396" deviceset="TP" device="-S2751-46R" value=""/>
+<part name="GND21" library="supply1" library_urn="urn:adsk.eagle:library:371" deviceset="GND" device=""/>
 </parts>
 <sheets>
@@
 <attribute name="VALUE" x="113.03" y="37.338" size="1.27" layer="96"/>
 </instance>
-<instance part="U$6" gate="G$1" x="15.24" y="13.97" smashed="yes"/>
+<instance part="U$6" gate="G$1" x="10.16" y="13.97" smashed="yes"/>
 <instance part="NFC" gate="G$1" x="72.39" y="40.005" smashed="yes" rot="MR0">
 <attribute name="VALUE" x="69.215" y="38.735" size="1.27" layer="96" rot="MR0"/>
@@
 <attribute name="NAME" x="188.595" y="165.735" size="1.778" layer="95" rot="R90"/>
 <attribute name="VALUE" x="188.595" y="151.13" size="1.778" layer="96" rot="R90"/>
+</instance>
+<instance part="X4" gate="X1" x="24.13" y="16.51" smashed="yes">
+<attribute name="NAME" x="21.59" y="22.86" size="1.778" layer="95"/>
+<attribute name="VALUE" x="21.59" y="20.32" size="1.778" layer="96"/>
+</instance>
+<instance part="X5" gate="X1" x="41.91" y="16.51" smashed="yes">
+<attribute name="NAME" x="39.37" y="22.86" size="1.778" layer="95"/>
+<attribute name="VALUE" x="39.37" y="20.32" size="1.778" layer="96"/>
+</instance>
+<instance part="X6" gate="X1" x="59.69" y="16.51" smashed="yes">
+<attribute name="NAME" x="57.15" y="22.86" size="1.778" layer="95"/>
+<attribute name="VALUE" x="57.15" y="20.32" size="1.778" layer="96"/>
+</instance>
+<instance part="U$2" gate="G$1" x="24.13" y="7.62" smashed="yes">
+<attribute name="VALUE" x="22.606" y="5.08" size="1.27" layer="96"/>
+</instance>
+<instance part="U$3" gate="G$1" x="41.91" y="7.62" smashed="yes">
+<attribute name="VALUE" x="40.386" y="5.08" size="1.27" layer="96"/>
+</instance>
+<instance part="U$4" gate="G$1" x="59.69" y="7.62" smashed="yes">
+<attribute name="VALUE" x="58.166" y="5.08" size="1.27" layer="96"/>
 </instance>
 </instances>
@@
 <wire x1="79.375" y1="45.72" x2="81.28" y2="45.72" width="0.1524" layer="91"/>
 </segment>
+<segment>
+<pinref part="X4" gate="X1" pin="C"/>
+<pinref part="U$2" gate="G$1" pin="GND"/>
+<wire x1="24.13" y1="11.43" x2="24.13" y2="10.16" width="0.1524" layer="91"/>
+</segment>
+<segment>
+<pinref part="X5" gate="X1" pin="C"/>
+<pinref part="U$3" gate="G$1" pin="GND"/>
+<wire x1="41.91" y1="10.16" x2="41.91" y2="11.43" width="0.1524" layer="91"/>
+</segment>
+<segment>
+<pinref part="X6" gate="X1" pin="C"/>
+<pinref part="U$4" gate="G$1" pin="GND"/>
+<wire x1="59.69" y1="10.16" x2="59.69" y2="11.43" width="0.1524" layer="91"/>
+</segment>
 </net>
 <net name="+3V3" class="0">
@@
 <attribute name="VALUE" x="143.51" y="74.295" size="1.27" layer="96"/>
 </instance>
-<instance part="GND15" gate="TP1" x="141.605" y="86.995" smashed="yes">
-<attribute name="NAME" x="142.24" y="91.44" size="1.778" layer="95" rot="R90"/>
-<attribute name="VALUE" x="140.97" y="91.44" size="1.778" layer="96"/>
-</instance>
-<instance part="GND17" gate="1" x="141.605" y="76.835" smashed="yes">
-<attribute name="VALUE" x="139.065" y="74.295" size="1.27" layer="96"/>
+<instance part="GND15" gate="TP1" x="135.255" y="86.995" smashed="yes">
+<attribute name="NAME" x="135.89" y="91.44" size="1.778" layer="95" rot="R90"/>
+<attribute name="VALUE" x="134.62" y="91.44" size="1.778" layer="96"/>
+</instance>
+<instance part="GND17" gate="1" x="135.255" y="76.835" smashed="yes">
+<attribute name="VALUE" x="132.715" y="74.295" size="1.27" layer="96"/>
 </instance>
 <instance part="R33" gate="G$1" x="53.975" y="77.47" smashed="yes">
@@
 <instance part="J6" gate="G$1" x="173.99" y="53.975" smashed="yes">
 <attribute name="NAME" x="172.72" y="71.755" size="1.778" layer="95"/>
+</instance>
+<instance part="GND18" gate="TP1" x="140.97" y="86.995" smashed="yes">
+<attribute name="NAME" x="141.605" y="91.44" size="1.778" layer="95" rot="R90"/>
+<attribute name="VALUE" x="140.335" y="91.44" size="1.778" layer="96"/>
+</instance>
+<instance part="GND21" gate="1" x="140.97" y="76.835" smashed="yes">
+<attribute name="VALUE" x="138.43" y="74.295" size="1.27" layer="96"/>
 </instance>
 </instances>
@@
 <segment>
 <pinref part="GND15" gate="TP1" pin="TP"/>
-<wire x1="141.605" y1="86.995" x2="141.605" y2="79.375" width="0.1524" layer="91"/>
+<wire x1="135.255" y1="86.995" x2="135.255" y2="79.375" width="0.1524" layer="91"/>
 <pinref part="GND17" gate="1" pin="GND"/>
 </segment>
@@
 <wire x1="32.385" y1="88.9" x2="26.67" y2="88.9" width="0.1524" layer="91"/>
 </segment>
-</net>
+<segment>
+<wire x1="140.97" y1="86.995" x2="140.97" y2="79.375" width="0.1524" layer="91"/>
+<pinref part="GND18" gate="TP1" pin="TP"/>
+<pinref part="GND21" gate="1" pin="GND"/>
+</segment>
+</net>

Commit message: update
1.Check the DRC again and remove the GND via short circuit bug
2.Modify the package and test point offset issue
Changed lines of the file:
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@@
 <drawing>
 <settings>
-<setting alwaysvectorfont="yes"/>
+<setting alwaysvectorfont="no"/>
 <setting verticaltext="up"/>
 </settings>
@@
 </segment>
 </net>
-<net name="VUSB_MCU" class="0">
-<segment>
-<wire x1="118.11" y1="106.68" x2="118.745" y2="106.68" width="0.1524" layer="91"/>
-</segment>
-</net>
