File: eagle/V1.0/M.2 SoM breakout board V1.0.brd (EAGLE design)
At the start: 140 x 122 mm, 119 parts, among them J1 3-PIN SMD, J11 WAFER-HY2.0-4PWB, J18 PARTICLE-STUDIOS_M_SERIES_M.2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, J2 DCJ0202, J21 SIP-2, J3 SPARK_CON_30X2_SMD, J5 SCREW-HOLE-3.7, J6 M.2-SOM-BREAKOUT-BOARD-V0.2-0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, J7 SCREW-HOLE-3.7, Q1 L2N7002, Q2 HSS2333, Q3 HSS2333, Q4 HSS2333, Q5 HSS2333, U1 XC8107, X1 BU-SMA-G, X2 BU-SMA-G, X3 BU-SMA-G, X4 S8111-46R, X5 S8111-46R, X6 S8111-46R

Commit message: Change Q2,Q3,Q4,Q5 value to SI2333DDS
Parts:
- Q2, Q3, Q4, Q5: value HSS2333 -> SI2333DS
Changed lines of the file:
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@@
 <attribute name="VALUE" x="26.6884" y="117.4282" size="1.778" layer="27"/>
 </element>
-<element name="Q4" library="RedBear" package="SOT-23" value="HSS2333" x="20.6568" y="97.0505" smashed="yes" rot="R270">
+<element name="Q4" library="RedBear" package="SOT-23" value="SI2333DS" x="20.6568" y="97.0505" smashed="yes" rot="R270">
 <attribute name="NAME" x="20.288" y="97.6455" size="0.8128" layer="51" rot="R270"/>
 <attribute name="VALUE" x="24.3534" y="92.8159" size="1.27" layer="27" rot="R90"/>
@@
 <attribute name="VALUE" value="100K" x="32.3152" y="110.6212" size="1" layer="27" rot="R270"/>
 </element>
-<element name="Q3" library="RedBear" package="SOT-23" value="HSS2333" x="35.535" y="105.87" smashed="yes" rot="R180">
+<element name="Q3" library="RedBear" package="SOT-23" value="SI2333DS" x="35.535" y="105.87" smashed="yes" rot="R180">
 <attribute name="NAME" x="36.3078" y="106.3912" size="0.8128" layer="51" rot="R180"/>
 <attribute name="VALUE" x="32.7302" y="104.741" size="1" layer="27"/>
 </element>
-<element name="Q5" library="RedBear" package="SOT-23" value="HSS2333" x="35.1384" y="109.188" smashed="yes" rot="R270">
+<element name="Q5" library="RedBear" package="SOT-23" value="SI2333DS" x="35.1384" y="109.188" smashed="yes" rot="R270">
 <attribute name="NAME" x="34.7188" y="109.8846" size="0.8128" layer="51" rot="R270"/>
 <attribute name="VALUE" x="34.4818" y="112.1198" size="1" layer="27" rot="R270"/>
@@
 <attribute name="VALUE" x="28.3069" y="108.2146" size="1" layer="27" rot="R90"/>
 </element>
-<element name="Q2" library="RedBear" package="SOT-23" value="HSS2333" x="17.7292" y="93.218" smashed="yes" rot="R90">
+<element name="Q2" library="RedBear" package="SOT-23" value="SI2333DS" x="17.7292" y="93.218" smashed="yes" rot="R90">
 <attribute name="NAME" x="18.8092" y="95.798" size="1" layer="25" rot="R90"/>
 <attribute name="VALUE" x="17.6492" y="95.798" size="1" layer="27" rot="R90"/>
